Commit message: Update joint limits of allegro

File: src/curobo/content/assets/robot/fr3_algr_zed2i/fr3_algr_zed2i.urdf (robot description, URDF)
Before this commit: robot fr3_algr, 40 links, 39 joints
Joints:
- joint algr_rh_if_axl: limit lower=-0.55 upper=0.55 effort=0.7 velocity=7 -> lower=-0.47 upper=0.47 effort=0.7 velocity=7
- joint algr_rh_if_dip: limit lower=-0.25 upper=1.72 effort=0.7 velocity=7 -> lower=-0.227 upper=1.618 effort=0.7 velocity=7
- joint algr_rh_if_mcp: limit lower=-0.25 upper=1.72 effort=0.7 velocity=7 -> lower=-0.196 upper=1.61 effort=0.7 velocity=7
- joint algr_rh_if_pip: limit lower=-0.25 upper=1.72 effort=0.7 velocity=7 -> lower=-0.174 upper=1.709 effort=0.7 velocity=7
- joint algr_rh_mf_axl: limit lower=-0.55 upper=0.55 effort=0.7 velocity=7 -> lower=-0.47 upper=0.47 effort=0.7 velocity=7
- joint algr_rh_mf_dip: limit lower=-0.25 upper=1.72 effort=0.7 velocity=7 -> lower=-0.227 upper=1.618 effort=0.7 velocity=7
- joint algr_rh_mf_mcp: limit lower=-0.25 upper=1.72 effort=0.7 velocity=7 -> lower=-0.196 upper=1.61 effort=0.7 velocity=7
- joint algr_rh_mf_pip: limit lower=-0.25 upper=1.72 effort=0.7 velocity=7 -> lower=-0.174 upper=1.709 effort=0.7 velocity=7
- joint algr_rh_rf_axl: limit lower=-0.55 upper=0.55 effort=0.7 velocity=7 -> lower=-0.47 upper=0.47 effort=0.7 velocity=7
- joint algr_rh_rf_dip: limit lower=-0.25 upper=1.72 effort=0.7 velocity=7 -> lower=-0.227 upper=1.618 effort=0.7 velocity=7
- joint algr_rh_rf_mcp: limit lower=-0.25 upper=1.72 effort=0.7 velocity=7 -> lower=-0.196 upper=1.61 effort=0.7 velocity=7
- joint algr_rh_rf_pip: limit lower=-0.25 upper=1.72 effort=0.7 velocity=7 -> lower=-0.174 upper=1.709 effort=0.7 velocity=7
- joint algr_rh_th_axl: limit lower=-0.3 upper=1.1 effort=0.7 velocity=7 -> lower=-0.105 upper=1.163 effort=0.7 velocity=7
- joint algr_rh_th_cmc: limit lower=0.263 upper=1.57 effort=0.7 velocity=7 -> lower=0.263 upper=1.396 effort=0.7 velocity=7
- joint algr_rh_th_ipl: limit lower=-0.1 upper=1.7 effort=0.7 velocity=7 -> lower=-0.162 upper=1.719 effort=0.7 velocity=7
- joint algr_rh_th_mcp: limit lower=-0.1 upper=1.71 effort=0.7 velocity=7 -> lower=-0.189 upper=1.644 effort=0.7 velocity=7
