Commit message: Add new iiwa 14 urdf, meshes, and update its config

File: src/curobo/content/assets/robot/iiwa_allegro_description/iiwa_allegro.urdf (robot description, URDF)
Before this commit: robot iiwa_allegro, 28 links, 27 joints
Links:
- removed link allegro_mount
- removed link base_link
- removed link iiwa7_link_0
- removed link iiwa7_link_1
- removed link iiwa7_link_2
- removed link iiwa7_link_3
- removed link iiwa7_link_4
- removed link iiwa7_link_5
- removed link iiwa7_link_6
- removed link iiwa7_link_7
- removed link iiwa7_link_ee
- added link allegro_custom_mount, mass 0.4375; collision mesh filename=new_mount_meshes/allegro-right-to-kuka-mount.stl scale=0.001 0.001 0.001; visual mesh filename=new_mount_meshes/allegro-right-to-kuka-mount.stl scale=0.001 0.001 0.001
- added link allegro_custom_mount2; collision mesh filename=new_mount_meshes/kuka_gopro_v2.stl scale=0.001 0.001 0.001; visual mesh filename=new_mount_meshes/kuka_gopro_v2.stl scale=0.001 0.001 0.001
- added link iiwa14_link_0, mass 5; collision mesh filename=new_iiwa14_meshes/collision/link_0.stl; visual mesh filename=new_iiwa14_meshes/visual/link_0.stl
- added link iiwa14_link_1, mass 4; collision mesh filename=new_iiwa14_meshes/collision/link_1.stl; visual mesh filename=new_iiwa14_meshes/visual/link_1.stl
- added link iiwa14_link_2, mass 4; collision mesh filename=new_iiwa14_meshes/collision/link_2.stl; visual mesh filename=new_iiwa14_meshes/visual/link_2.stl
- added link iiwa14_link_2_sphere2
- added link iiwa14_link_2_sphere3
- added link iiwa14_link_2_sphere4
- added link iiwa14_link_3, mass 3; collision mesh filename=new_iiwa14_meshes/collision/link_3.stl; visual mesh filename=new_iiwa14_meshes/visual/link_3.stl
- added link iiwa14_link_4, mass 2.7; collision mesh filename=new_iiwa14_meshes/collision/link_4.stl; visual mesh filename=new_iiwa14_meshes/visual/link_4.stl
- added link iiwa14_link_4_sphere2
- added link iiwa14_link_4_sphere3
- added link iiwa14_link_5, mass 1.7; collision mesh filename=new_iiwa14_meshes/collision/link_5.stl; visual mesh filename=new_iiwa14_meshes/visual/link_5.stl
- added link iiwa14_link_6, mass 1.8; collision mesh filename=new_iiwa14_meshes/collision/link_6.stl; visual mesh filename=new_iiwa14_meshes/visual/link_6.stl
- added link iiwa14_link_6_sphere2
- added link iiwa14_link_6_sphere3
- added link iiwa14_link_7, mass 0.3; collision mesh filename=new_iiwa14_meshes/collision/link_7.stl; visual mesh filename=new_iiwa14_meshes/visual/link_7.stl
- added link iiwa14_link_ee
- added link index_biotac_tip, mass 0.0168; collision sphere radius=0.012; visual mesh filename=new_allegro_meshes/link_3.0_tip.STL
- added link index_link_1_sphere2
- added link index_link_2_sphere2
- added link index_link_3_sphere2
- added link middle_biotac_tip, mass 0.0168; collision sphere radius=0.012; visual mesh filename=new_allegro_meshes/link_3.0_tip.STL
- added link middle_link_1_sphere2
- added link middle_link_2_sphere2
- added link middle_link_3_sphere2
- added link palm_link_content, mass 0.4154; collision box size=0.0408 0.1130 0.095; visual mesh filename=new_allegro_meshes/base_link.STL
- added link palm_link_sphere2
- added link palm_link_sphere3
- added link palm_link_sphere4
- added link palm_link_sphere5
- added link palm_link_sphere6
- added link palm_link_sphere7
- added link palm_link_sphere8
- added link palm_link_sphere9
- added link palm_x, mass 0.04
- added link palm_x_neg, mass 0.04
- added link palm_y, mass 0.04
- added link palm_y_neg, mass 0.04
- added link palm_z, mass 0.04
- added link palm_z_neg, mass 0.04
- added link ring_biotac_tip, mass 0.0168; collision sphere radius=0.012; visual mesh filename=new_allegro_meshes/link_3.0_tip.STL
- added link ring_link_1_sphere2
- added link ring_link_2_sphere2
- added link ring_link_3_sphere2
- added link thumb_biotac_tip, mass 0.0168; collision sphere radius=0.012; visual mesh filename=new_allegro_meshes/link_15.0_tip.STL
- added link thumb_link_2_sphere2
- added link thumb_link_3_sphere2
- added link thumb_link_3_sphere3
- link index_link_0: mass 0.005 -> 0.0119; geometry collision box size=0.0196 0.0275 0.0164; visual mesh filename=new_allegro_meshes/link_0.0.STL
- link index_link_1: mass 0.125164 -> 0.065; geometry collision box size=0.0196 0.0275 0.054; visual mesh filename=new_allegro_meshes/link_1.0.STL
- link index_link_2: mass 0.131691 -> 0.0355; geometry collision box size=0.0196 0.0275 0.0384; visual mesh filename=new_allegro_meshes/link_2.0.STL
- link index_link_3: mass 0.0211922 -> 0.0096; geometry collision box size=0.0196 0.0275 0.0267; visual mesh filename=new_allegro_meshes/link_3.0.STL
- link middle_link_0: mass 0.005 -> 0.0119; geometry collision box size=0.0196 0.0275 0.0164; visual mesh filename=new_allegro_meshes/link_0.0.STL
- link middle_link_1: mass 0.125164 -> 0.065; geometry collision box size=0.0196 0.0275 0.054; visual mesh filename=new_allegro_meshes/link_1.0.STL
- link middle_link_2: mass 0.131691 -> 0.0355; geometry collision box size=0.0196 0.0275 0.0384; visual mesh filename=new_allegro_meshes/link_2.0.STL
- link middle_link_3: mass 0.0211922 -> 0.0096; geometry collision box size=0.0196 0.0275 0.0267; visual mesh filename=new_allegro_meshes/link_3.0.STL
- link palm_link: mass 0.4154 -> None; geometry 
- link ring_link_0: mass 0.005 -> 0.0119; geometry collision box size=0.0196 0.0275 0.0164; visual mesh filename=new_allegro_meshes/link_0.0.STL
- link ring_link_1: mass 0.125164 -> 0.065; geometry collision box size=0.0196 0.0275 0.054; visual mesh filename=new_allegro_meshes/link_1.0.STL
- link ring_link_2: mass 0.131691 -> 0.0355; geometry collision box size=0.0196 0.0275 0.0384; visual mesh filename=new_allegro_meshes/link_2.0.STL
- link ring_link_3: mass 0.0211922 -> 0.0096; geometry collision box size=0.0196 0.0275 0.0267; visual mesh filename=new_allegro_meshes/link_3.0.STL
- link thumb_link_0: mass 0.1 -> 0.0176; geometry collision box size=0.0358 0.034 0.0455; visual mesh filename=new_allegro_meshes/link_12.0_right.STL
- link thumb_link_1: mass 0.1 -> 0.0119; geometry collision box size=0.0196 0.0275 0.0177; visual mesh filename=new_allegro_meshes/link_13.0.STL
- link thumb_link_2: mass 0.1 -> 0.038; geometry collision box size=0.0196 0.0275 0.0514; visual mesh filename=new_allegro_meshes/link_14.0.STL
- link thumb_link_3: mass 0.1 -> 0.0388; geometry collision box size=0.0196 0.0275 0.0423; visual mesh filename=new_allegro_meshes/link_15.0.STL
Joints:
- removed joint allegro_mount_joint
- removed joint iiwa7_allegro
- removed joint iiwa7_base_link_iiwa7_joint
- removed joint iiwa7_joint_1
- removed joint iiwa7_joint_2
- removed joint iiwa7_joint_3
- removed joint iiwa7_joint_4
- removed joint iiwa7_joint_5
- removed joint iiwa7_joint_6
- removed joint iiwa7_joint_7
- removed joint iiwa7_joint_ee
- added joint iiwa14_allegro: type fixed, parent iiwa14_link_ee, child palm_link, origin xyz=-0.14 0 0.0325 rpy=0 -1.57 0
- added joint iiwa14_allegro_custom_mount: type fixed, parent iiwa14_link_ee, child allegro_custom_mount, origin xyz=-0.0128878 0.0562605 0.006 rpy=0 0 1.57
- added joint iiwa14_allegro_custom_mount2: type fixed, parent iiwa14_link_ee, child allegro_custom_mount2, origin xyz=0 0 0.006 rpy=3.14 0 -1.57
- added joint iiwa14_joint_1: type revolute, parent iiwa14_link_0, child iiwa14_link_1, origin xyz=0 0 0.1575 rpy=0 0 0, axis 0 0 1, limit lower=-2.96705972839 upper=2.96705972839 effort=300 velocity=10
- added joint iiwa14_joint_2: type revolute, parent iiwa14_link_1, child iiwa14_link_2, origin xyz=0 0 0.2025 rpy=1.57079632679   0 3.14159265359, axis 0 0 1, limit lower=-2.09439510239 upper=2.09439510239 effort=300 velocity=10
- added joint iiwa14_joint_2_sphere2: type fixed, parent iiwa14_link_2, child iiwa14_link_2_sphere2, origin xyz=0 0.15 0 rpy=0 0 0, axis 0 0 1
- added joint iiwa14_joint_2_sphere3: type fixed, parent iiwa14_link_2, child iiwa14_link_2_sphere3, origin xyz=0 0.25 0 rpy=0 0 0, axis 0 0 1
- added joint iiwa14_joint_2_sphere4: type fixed, parent iiwa14_link_2, child iiwa14_link_2_sphere4, origin xyz=0 -0.25 0 rpy=0 0 0, axis 0 0 1
- added joint iiwa14_joint_3: type revolute, parent iiwa14_link_2, child iiwa14_link_3, origin xyz=0 0.2045 0 rpy=1.57079632679 0 3.14159265359, axis 0 0 1, limit lower=-2.96705972839 upper=2.96705972839 effort=300 velocity=10
- added joint iiwa14_joint_4: type revolute, parent iiwa14_link_3, child iiwa14_link_4, origin xyz=0 0 0.2155 rpy=1.57079632679 0 0, axis 0 0 1, limit lower=-2.09439510239 upper=2.09439510239 effort=300 velocity=10
- added joint iiwa14_joint_4_sphere2: type fixed, parent iiwa14_link_4, child iiwa14_link_4_sphere2, origin xyz=0 0.15 0 rpy=0 0 0, axis 0 0 1
- added joint iiwa14_joint_4_sphere3: type fixed, parent iiwa14_link_4, child iiwa14_link_4_sphere3, origin xyz=0 0.25 0 rpy=0 0 0, axis 0 0 1
- added joint iiwa14_joint_5: type revolute, parent iiwa14_link_4, child iiwa14_link_5, origin xyz=0 0.1845 0 rpy=-1.57079632679 3.14159265359 0, axis 0 0 1, limit lower=-2.96705972839 upper=2.96705972839 effort=300 velocity=10
- added joint iiwa14_joint_6: type revolute, parent iiwa14_link_5, child iiwa14_link_6, origin xyz=0 0 0.2155 rpy=1.57079632679 0 0, axis 0 0 1, limit lower=-2.09439510239 upper=2.09439510239 effort=300 velocity=10
- added joint iiwa14_joint_6_sphere2: type fixed, parent iiwa14_link_6, child iiwa14_link_6_sphere2, origin xyz=0 0 0 rpy=0 0 0, axis 0 0 1
- added joint iiwa14_joint_6_sphere3: type fixed, parent iiwa14_link_6, child iiwa14_link_6_sphere3, origin xyz=0 0 -0.05 rpy=0 0 0, axis 0 0 1
- added joint iiwa14_joint_7: type revolute, parent iiwa14_link_6, child iiwa14_link_7, origin xyz=0 0.081 0 rpy=-1.57079632679 3.14159265359 0, axis 0 0 1, limit lower=-3.05432619099 upper=3.05432619099 effort=300 velocity=10
- added joint iiwa14_joint_ee: type fixed, parent iiwa14_link_7, child iiwa14_link_ee, origin xyz=0 0 0.045 rpy=0 0 0
- added joint index_biotac_tip_joint: type fixed, parent index_link_3, child index_biotac_tip, origin xyz=0 0 0.0267 rpy=0 0 0
- added joint index_link_1_joint_sphere2: type fixed, parent index_link_1, child index_link_1_sphere2, origin xyz=0.0 0.0 0.027 rpy=0 0 0, axis 0 0 1
- added joint index_link_2_joint_sphere2: type fixed, parent index_link_2, child index_link_2_sphere2, origin xyz=0.0 0.0 0.027 rpy=0 0 0, axis 0 0 1
- added joint index_link_3_joint_sphere2: type fixed, parent index_link_3, child index_link_3_sphere2, origin xyz=0.0 0.0 0.027 rpy=0 0 0, axis 0 0 1
- added joint middle_biotac_tip_joint: type fixed, parent middle_link_3, child middle_biotac_tip, origin xyz=0 0 0.0267 rpy=0 0 0
- added joint middle_link_1_joint_sphere2: type fixed, parent middle_link_1, child middle_link_1_sphere2, origin xyz=0.0 0.0 0.027 rpy=0 0 0, axis 0 0 1
- added joint middle_link_2_joint_sphere2: type fixed, parent middle_link_2, child middle_link_2_sphere2, origin xyz=0.0 0.0 0.027 rpy=0 0 0, axis 0 0 1
- added joint middle_link_3_joint_sphere2: type fixed, parent middle_link_3, child middle_link_3_sphere2, origin xyz=0.0 0.0 0.027 rpy=0 0 0, axis 0 0 1
- added joint palm_link_joint_content: type fixed, parent palm_link, child palm_link_content, origin xyz=0 0 0 rpy=0 0 0
- added joint palm_link_joint_sphere2: type fixed, parent palm_link, child palm_link_sphere2, origin xyz=-0.02 0.03 -0.03 rpy=0 0 0, axis 0 0 1
- added joint palm_link_joint_sphere3: type fixed, parent palm_link, child palm_link_sphere3, origin xyz=-0.02 -0.03 -0.03 rpy=0 0 0, axis 0 0 1
- added joint palm_link_joint_sphere4: type fixed, parent palm_link, child palm_link_sphere4, origin xyz=-0.02 0.03 -0.1 rpy=0 0 0, axis 0 0 1
- added joint palm_link_joint_sphere5: type fixed, parent palm_link, child palm_link_sphere5, origin xyz=-0.02 -0.03 -0.1 rpy=0 0 0, axis 0 0 1
- added joint palm_link_joint_sphere6: type fixed, parent palm_link, child palm_link_sphere6, origin xyz=-0.02 0.03 -0.17 rpy=0 0 0, axis 0 0 1
- added joint palm_link_joint_sphere7: type fixed, parent palm_link, child palm_link_sphere7, origin xyz=-0.02 -0.03 -0.17 rpy=0 0 0, axis 0 0 1
- added joint palm_link_joint_sphere8: type fixed, parent palm_link, child palm_link_sphere8, origin xyz=-0.02 -0.08 -0.12 rpy=0 0 0, axis 0 0 1
- added joint palm_link_joint_sphere9: type fixed, parent palm_link, child palm_link_sphere9, origin xyz=0.03 -0.08 -0.12 rpy=0 0 0, axis 0 0 1
- added joint palm_x_joint: type fixed, parent palm_link, child palm_x, origin xyz=0.25 0. 0. rpy=0. 0. 0.
- added joint palm_x_neg_joint: type fixed, parent palm_link, child palm_x_neg, origin xyz=-0.25 0. 0. rpy=0. 0. 0.
- added joint palm_y_joint: type fixed, parent palm_link, child palm_y, origin xyz=0. 0.25 0. rpy=0. 0. 0.
- added joint palm_y_neg_joint: type fixed, parent palm_link, child palm_y_neg, origin xyz=0. -0.25 0. rpy=0. 0. 0.
- added joint palm_z_joint: type fixed, parent palm_link, child palm_z, origin xyz=0. 0. 0.25 rpy=0. 0. 0.
- added joint palm_z_neg_joint: type fixed, parent palm_link, child palm_z_neg, origin xyz=0. 0. -0.25 rpy=0. 0. 0.
- added joint ring_biotac_tip_joint: type fixed, parent ring_link_3, child ring_biotac_tip, origin xyz=0 0 0.0267 rpy=0 0 0
- added joint ring_link_1_joint_sphere2: type fixed, parent ring_link_1, child ring_link_1_sphere2, origin xyz=0.0 0.0 0.027 rpy=0 0 0, axis 0 0 1
- added joint ring_link_2_joint_sphere2: type fixed, parent ring_link_2, child ring_link_2_sphere2, origin xyz=0.0 0.0 0.027 rpy=0 0 0, axis 0 0 1
- added joint ring_link_3_joint_sphere2: type fixed, parent ring_link_3, child ring_link_3_sphere2, origin xyz=0.0 0.0 0.027 rpy=0 0 0, axis 0 0 1
- added joint thumb_biotac_tip_joint: type fixed, parent thumb_link_3, child thumb_biotac_tip, origin xyz=0 0 0.0423 rpy=0 0 0
- added joint thumb_link_2_joint_sphere2: type fixed, parent thumb_link_2, child thumb_link_2_sphere2, origin xyz=0.0 0.0 0.025 rpy=0 0 0, axis 0 0 1
- added joint thumb_link_3_joint_sphere2: type fixed, parent thumb_link_3, child thumb_link_3_sphere2, origin xyz=0.0 0.0 0.025 rpy=0 0 0, axis 0 0 1
- added joint thumb_link_3_joint_sphere3: type fixed, parent thumb_link_3, child thumb_link_3_sphere3, origin xyz=0.0 0.0 0.055 rpy=0 0 0, axis 0 0 1
- joint index_joint_0: limit lower=-0.558488888889 upper=0.558488888889 effort=0.35 velocity=6.283 -> lower=-0.47 upper=0.47 effort=15 velocity=7; origin xyz=0.0514302 -0.03632 -0.0113 rpy=3.1415 -1.57075 -0.0872638888889 -> xyz=0 0.0435 -0.001542 rpy=-0.08726646255 0 0
- joint index_joint_1: axis 0 0 1 -> 0 1 0; limit lower=-0.279244444444 upper=1.727825 effort=0.35 velocity=6.283 -> lower=-0.196 upper=1.61 effort=15 velocity=7; origin xyz=0.0 0.0 0.0 rpy=3.1415 -1.57075 1.57075 -> xyz=0 0 0.0164
- joint index_joint_2: axis 0 0 1 -> 0 1 0; limit lower=-0.279244444444 upper=1.727825 effort=0.35 velocity=6.283 -> lower=-0.174 upper=1.709 effort=15 velocity=7; origin xyz=0.054 0.0 0.0 rpy=0.0 0.0 0.0 -> xyz=0 0 0.054
- joint index_joint_3: axis 0 0 1 -> 0 1 0; limit lower=-0.279244444444 upper=1.727825 effort=0.35 velocity=6.283 -> lower=-0.227 upper=1.618 effort=15 velocity=7; origin xyz=0.0384 0.0 0.0 rpy=0.0 0.0 0.0 -> xyz=0 0 0.0384
- joint middle_joint_0: limit lower=-0.558488888889 upper=0.558488888889 effort=0.35 velocity=6.283 -> lower=-0.47 upper=0.47 effort=15 velocity=7; origin xyz=0.0537375 0.0087771 -0.0113 rpy=3.1415 -1.57075 0 -> xyz=0 0 0.0007 rpy=0.0 0 0
- joint middle_joint_1: axis 0 0 1 -> 0 1 0; limit lower=-0.279244444444 upper=1.727825 effort=0.35 velocity=6.283 -> lower=-0.196 upper=1.61 effort=15 velocity=7; origin xyz=0.0 0.0 0.0 rpy=3.1415 -1.57075 1.57075 -> xyz=0 0 0.0164
- joint middle_joint_2: axis 0 0 1 -> 0 1 0; limit lower=-0.279244444444 upper=1.727825 effort=0.35 velocity=6.283 -> lower=-0.174 upper=1.709 effort=15 velocity=7; origin xyz=0.054 0.0 0.0 rpy=0.0 0.0 0.0 -> xyz=0 0 0.054
- joint middle_joint_3: axis 0 0 1 -> 0 1 0; limit lower=-0.279244444444 upper=1.727825 effort=0.35 velocity=6.283 -> lower=-0.227 upper=1.618 effort=15 velocity=7; origin xyz=0.0384 0.0 0.0 rpy=0.0 0.0 0.0 -> xyz=0 0 0.0384
- joint ring_joint_0: limit lower=-0.558488888889 upper=0.558488888889 effort=0.35 velocity=6.283 -> lower=-0.47 upper=0.47 effort=15 velocity=7; origin xyz=0.0514302 0.0538749 -0.0113 rpy=3.1415 -1.57075 0.0872638888889 -> xyz=0 -0.0435 -0.001542 rpy=0.08726646255 0 0
- joint ring_joint_1: axis 0 0 1 -> 0 1 0; limit lower=-0.279244444444 upper=1.727825 effort=0.35 velocity=6.283 -> lower=-0.196 upper=1.61 effort=15 velocity=7; origin xyz=0.0 0.0 0.0 rpy=3.1415 -1.57075 1.57075 -> xyz=0 0 0.0164
- joint ring_joint_2: axis 0 0 1 -> 0 1 0; limit lower=-0.279244444444 upper=1.727825 effort=0.35 velocity=6.283 -> lower=-0.174 upper=1.709 effort=15 velocity=7; origin xyz=0.054 0.0 0.0 rpy=0.0 0.0 0.0 -> xyz=0 0 0.054
- joint ring_joint_3: axis 0 0 1 -> 0 1 0; limit lower=-0.279244444444 upper=1.727825 effort=0.35 velocity=6.283 -> lower=-0.227 upper=1.618 effort=15 velocity=7; origin xyz=0.0384 0.0 0.0 rpy=0.0 0.0 0.0 -> xyz=0 0 0.0384
- joint thumb_joint_0: axis 0 0 1 -> -1 0 0; limit lower=0.279244444444 upper=1.57075 effort=0.35 velocity=6.283 -> lower=0.263 upper=1.396 effort=15 velocity=7; origin xyz=-0.0367482 -0.0081281 -0.0295 rpy=-1.57075 -1.57075 1.48348611111 -> xyz=-0.0182 0.019333 -0.045987 rpy=0 -1.65806278845 -1.5707963259
- joint thumb_joint_1: limit lower=-0.331602777778 upper=1.15188333333 effort=0.35 velocity=6.283 -> lower=-0.105 upper=1.163 effort=15 velocity=7; origin xyz=0.005 0.0 0.0 rpy=1.57075 0 0 -> xyz=-0.027 0.005 0.0399
- joint thumb_joint_2: axis 0 0 1 -> 0 1 0; limit lower=-0.279244444444 upper=1.727825 effort=0.35 velocity=6.283 -> lower=-0.189 upper=1.644 effort=15 velocity=7; origin xyz=0 0 0.0554 rpy=3.1415 -1.57075 0.0 -> xyz=0 0 0.0177
- joint thumb_joint_3: axis 0 0 1 -> 0 1 0; limit lower=-0.279244444444 upper=1.76273055556 effort=0.35 velocity=6.283 -> lower=-0.162 upper=1.719 effort=15 velocity=7; origin xyz=0.0514 0.0 0.0 rpy=0.0 0.0 0.0 -> xyz=0 0 0.0514
