Commit message: Add updated bimanual kuka allegro assets

File: src/curobo/content/assets/robot/bimanual_kuka_allegro/bimanual_kuka_allegro_ORIGNIAL.urdf (robot description, URDF)
Before this commit: robot bimanual_kuka_allegro, 127 links, 126 joints
Joints:
- joint left_index_joint_0: origin xyz=0 -0.0435 -0.001542 rpy=0.08726646255 0 0 -> xyz=0 0.0435 -0.001542 rpy=-0.08726646255 0 0
- joint left_ring_joint_0: origin xyz=0 0.0435 -0.001542 rpy=-0.08726646255 0 0 -> xyz=0 -0.0435 -0.001542 rpy=0.08726646255 0 0
